Commit message: main_frame design edits made

File: install/swarm/share/swarm/model/main_frame.xacro (robot description, xacro)
@@ -65,4 +65,16 @@
     <collision name="lidar_scan_collision">
     <origin xyz="0.424 0 0.327" rpy="0 0 0"/>
+    <geometry>
+      <box size="0.0078 0.13 0.0192"/>
+    </geometry>
+  </collision>
+      <collision name="user_rail_collision">
+    <origin xyz="0.272 0 0.245" rpy="0 0 0"/>
+    <geometry>
+      <box size="0.0078 0.13 0.0192"/>
+    </geometry>
+  </collision>
+      <collision name="holder_collision">
+    <origin xyz="0.272 0 0.245" rpy="0 0 0"/>
     <geometry>
       <box size="0.0078 0.13 0.0192"/>
@@ -140,4 +152,22 @@
   </geometry>
   </visual>
+      <visual name="user_rail_visual">
+  <origin xyz="0.272 0 0.245" rpy="0 0 0"/>
+  <geometry>
+  	<mesh filename="package://swarm/meshes/user_rail.dae" scale="1 1 1"/>
+  </geometry>
+  <material name="black">
+  	<color rgba="0.1 0.1 0.1 1"/>
+  </material>
+  </visual>
+        <visual name="holder_visual">
+  <origin xyz="0.272 0 0" rpy="0 0 0"/>
+  <geometry>
+  	<mesh filename="package://swarm/meshes/holder.stl" scale="1 1 1"/>
+  </geometry>
+  <material name="black">
+  	<color rgba="0.1 0.1 0.1 1"/>
+  </material>
+  </visual>
 </link>
 <joint name="base_link_joint" type="fixed">

File: install/swarm/share/swarm/model/robot.xacro (robot description, xacro)
@@ -5,3 +5,14 @@
   <xacro:include filename="$(find swarm)/model/wheels.xacro"/>
   <xacro:wheels/>
+  <xacro:include filename="cameras.xacro"/>
+  <xacro:depth_camera
+    name="front_camera_link"
+    parent="ground_bot_frame"
+    xyz="0.478 0 0.285"
+    rpy="0 0 0"/>
+  <xacro:depth_camera
+    name="down_camera_link"
+    parent="ground_bot_frame"
+    xyz="0.478 0 0.200"
+    rpy="0 0.5236 0"/>
 </robot>
