Commit message: ROS topics established and drone files added

File: src/swarm/model/ground_bot.xacro (robot description, xacro)
@@ -1,5 +1,5 @@
 <?xml version="1.9"?>
 <robot xmlns:xacro="http://www.ros.org/wiki/xacro">
-  <xacro:macro name="bot">
+  <xacro:macro name="ground_bot">
     <link name="base_link"/>
     <link name="ground_bot_frame">
@@ -95,5 +95,5 @@
     </joint>
     <gazebo reference="ground_bot_frame">
-      <sensor name="imu_sensor" type="imu">
+      <sensor name="imu" type="imu">
         <always_on>true</always_on>
         <update_rate>100</update_rate>

File: src/swarm/model/lidar.xacro (robot description, xacro)
@@ -4,5 +4,5 @@
     <link name="${name}">
       <visual name="lidar_base_visual_2">
-        <origin xyz="0.424 0 0.327" rpy="0 0 0"/>
+        <origin xyz="0 0 0" rpy="0 0 0"/>
         <geometry>
           <mesh
@@ -12,5 +12,5 @@
       </visual>
       <visual name="lidar_base_visual">
-        <origin xyz="0.424 0 0.327" rpy="0 0 0"/>
+        <origin xyz="0 0 0" rpy="0 0 0"/>
         <geometry>
           <mesh
@@ -28,5 +28,5 @@
       </visual>
       <collision name="lidar_base_collision">
-        <origin xyz="0.424 0 0.327" rpy="0 0 0"/>
+        <origin xyz="0.212 0 0.164" rpy="0 0 0"/>
         <geometry>
           <box size="0.0078 0.13 0.0192"/>
@@ -34,5 +34,5 @@
       </collision>
       <collision name="lidar_base_collision_2">
-        <origin xyz="0.424 0 0.327" rpy="0 0 0"/>
+        <origin xyz="0.212 0 0.164" rpy="0 0 0"/>
         <geometry>
           <mesh size="0.0078 0.13 0.0192"/>

File: src/swarm/model/robot.xacro (robot description, xacro)
@@ -3,7 +3,11 @@
   xmlns:xacro="http://www.ros.org/wiki/xacro"
   name="Ground_bot">
-  <!-- Main frame -->
-  <xacro:include filename="$(find swarm)/model/main_frame.xacro"/>
-  <xacro:bot/>
+  <xacro:include filename="$(find swarm)/model/robot.gazebo"/>
+  <!-- Ground Bot -->
+  <xacro:include filename="$(find swarm)/model/ground_bot.xacro"/>
+  <xacro:ground_bot/>
+    <!-- Drone
+  <xacro:include filename="$(find swarm)/model/drone.xacro"/>
+-->
   <!-- Wheels -->
   <xacro:include filename="$(find swarm)/model/wheels.xacro"/>
@@ -16,9 +20,4 @@
     xyz="0.478 0 0.285"
     rpy="0 0 0"/>
-  <xacro:depth_camera
-    name="down_camera"
-    parent="ground_bot_frame"
-    xyz="0.478 0 0.200"
-    rpy="0 0.5236 0"/>
   <!-- LiDAR -->
   <xacro:include filename="$(find swarm)/model/lidar.xacro"/>
