Commit message: Bot binary movement sorted

File: src/swarm/model/wheels.xacro (robot description, xacro)
@@ -42,5 +42,5 @@
       <child link="front_left_wheel"/>
       <origin xyz="0.256 0.2854 0.03282" rpy="0 0 0"/>
-      <axis xyz="1 0 0"/>
+      <axis xyz="0 1 0"/>
       <limit lower="-1e16" upper="1e16" effort="20" velocity="50"/>
     </joint>
@@ -49,5 +49,5 @@
       <child link="front_right_wheel"/>
       <origin xyz="0.256 -0.2854 0.03282" rpy="0 0 0"/>
-      <axis xyz="1 0 0"/>
+      <axis xyz="0 1 0"/>
       <limit lower="-1e16" upper="1e16" effort="20" velocity="50"/>
     </joint>
@@ -56,5 +56,5 @@
       <child link="rear_left_wheel"/>
       <origin xyz="-0.256 0.2854 0.03282" rpy="0 0 0"/>
-      <axis xyz="1 0 0"/>
+      <axis xyz="0 1 0"/>
       <limit lower="-1e16" upper="1e16" effort="20" velocity="50"/>
     </joint>
@@ -63,5 +63,5 @@
       <child link="rear_right_wheel"/>
       <origin xyz="-0.256 -0.2854 0.03282" rpy="0 0 0"/>
-      <axis xyz="1 0 0"/>
+      <axis xyz="0 1 0"/>
       <limit lower="-1e16" upper="1e16" effort="20" velocity="50"/>
     </joint>
