Commit message: corrective changes in robot configuartion

File: src/swarm/model/cameras.xacro (robot description, xacro)
@@ -1,3 +1,3 @@
-<?xml version="1.0"?>
+<?xml version="1.9"?>
 <robot xmlns:xacro="http://www.ros.org/wiki/xacro">
   <xacro:macro name="depth_camera" params="name parent xyz rpy">

File: src/swarm/model/main_frame.xacro (robot description, xacro)
@@ -1,188 +1,105 @@
-<?xml version="1.0"?>
+<?xml version="1.9"?>
 <robot xmlns:xacro="http://www.ros.org/wiki/xacro">
-<xacro:macro name="bot">
-<link name="base_link"/>
-<link name="ground_bot_frame">
-  <inertial>
-    <origin xyz="0.0 0.0 -0.25" rpy="0 0 0"/>
-    <mass value="40.0"/>
-    <inertia
-        ixx="0.615397"
-        ixy="-0.0240585"
-        ixz="-0.120749"
-        iyy="1.75388"
-        iyz="-0.0028322"
-        izz="2.03641"/>
-  </inertial>
-  <collision name="main_frame_collision">
-    <origin xyz="0 0 0.12" rpy="0 0 0"/>
-    <geometry>
-      <box size="0.9874 0.5709 0.05"/>
-    </geometry>
-  </collision>
-  <collision name="frame_bottom_collision">
-    <origin xyz="0 0 0.046" rpy="0 0 0"/>
-    <geometry>
-      <box size="0.80 0.5709 0.095"/>
-    </geometry>
-  </collision>
-  <collision name="frame_collision_1">
-    <origin xyz="0 0 0.185625" rpy="0 0 0"/>
-    <geometry>
-      <box size="0.78992 0.5709 0.12375"/>
-    </geometry>
-  </collision>
-  <collision name="front_camera_collision">
-    <origin xyz="0.478 0 0.285" rpy="0 0 0"/>
-    <geometry>
-      <box size="0.0078 0.13 0.0192"/>
-    </geometry>
-  </collision>
-  <collision name="down_camera_collision">
-    <origin xyz="0.473 0 0.260" rpy="0 0.5236 0"/>
-    <geometry>
-      <box size="0.0078 0.13 0.0192"/>
-    </geometry>
-  </collision>
-    <collision name="top_chassis_collision">
-    <origin xyz="0 0 0" rpy="0 0 0"/>
-    <geometry>
-      <box size="0.0078 0.13 0.0192"/>
-    </geometry>
-  </collision>
-  <collision name="lidar_base_collision">
-    <origin xyz="0.424 0 0.327" rpy="0 0 0"/>
-    <geometry>
-      <box size="0.0078 0.13 0.0192"/>
-    </geometry>
-  </collision>
-  <collision name="lidar_base_collision_2">
-    <origin xyz="0.424 0 0.327" rpy="0 0 0"/>
-    <geometry>
-      <box size="0.0078 0.13 0.0192"/>
-    </geometry>
-  </collision>
-    <collision name="lidar_scan_collision">
-    <origin xyz="0.424 0 0.327" rpy="0 0 0"/>
-    <geometry>
-      <box size="0.0078 0.13 0.0192"/>
-    </geometry>
-  </collision>
+  <xacro:macro name="bot">
+    <link name="base_link"/>
+    <link name="ground_bot_frame">
+      <inertial>
+        <origin xyz="0.0 0.0 -0.25" rpy="0 0 0"/>
+        <mass value="40.0"/>
+        <inertia
+          ixx="0.615397"
+          ixy="-0.0240585"
+          ixz="-0.120749"
+          iyy="1.75388"
+          iyz="-0.0028322"
+          izz="2.03641"/>
+      </inertial>
+      <collision name="main_frame_collision">
+        <origin xyz="0 0 0.12" rpy="0 0 0"/>
+        <geometry>
+          <box size="0.9874 0.5709 0.05"/>
+        </geometry>
+      </collision>
+      <collision name="frame_bottom_collision">
+        <origin xyz="0 0 0.046" rpy="0 0 0"/>
+        <geometry>
+          <box size="0.80 0.5709 0.095"/>
+        </geometry>
+      </collision>
+      <collision name="frame_collision_1">
+        <origin xyz="0 0 0.185625" rpy="0 0 0"/>
+        <geometry>
+          <box size="0.78992 0.5709 0.12375"/>
+        </geometry>
+      </collision>
+            <collision name="top_chassis_collision">
+        <origin xyz="0 0 0" rpy="0 0 0"/>
+        <geometry>
+          <box size="0.0078 0.13 0.0192"/>
+        </geometry>
+      </collision>
       <collision name="user_rail_collision">
-    <origin xyz="0.272 0 0.245" rpy="0 0 0"/>
-    <geometry>
-      <box size="0.0078 0.13 0.0192"/>
-    </geometry>
-  </collision>
-      <collision name="holder_collision">
-    <origin xyz="0.272 0 0.245" rpy="0 0 0"/>
-    <geometry>
-      <box size="0.0078 0.13 0.0192"/>
-    </geometry>
-  </collision>
-  <visual name="main_frame_visual">
-    <geometry>
-      <mesh filename="package://swarm/meshes/main_frame.stl" scale="1 1 1"/>
-    </geometry>
-    <material name="black">
+        <origin xyz="0.272 0 0.245" rpy="0 0 0"/>
+        <geometry>
+          <box size="0.0078 0.13 0.0192"/>
+        </geometry>
+      </collision>
+      <visual name="main_frame_visual">
+        <geometry>
+          <mesh filename="package://swarm/meshes/main_frame.stl"/>
+        </geometry>
+        <material name="black">
           <color rgba="0.1 0.1 0.1 1"/>
         </material>
-  </visual>
-  <visual name="down_camera_visual">
-    <origin xyz="0.478 0 0.200" rpy="0 0.5236 0"/>
-    <geometry>
-      <mesh filename="package://swarm/meshes/zed2i.stl" scale="1 1 1"/>
-    </geometry>
-    <material name="black">
-          <color rgba="0.1 0.1 0.1 1"/>
-    </material>
-  </visual>
-  <visual name="front_camera_visual">
-    <origin xyz="0.478 0 0.285" rpy="0 0 0"/>
-    <geometry>
-      <mesh filename="package://swarm/meshes/zed2i.stl" scale="1 1 1"/>
-    </geometry>
-    <material name="black">
-          <color rgba="0.1 0.1 0.1 1"/>
-    </material>
-  </visual>
-  <visual name="front_bumper_visual">
-    <origin xyz="0.48 0 0.091" rpy="0 0 0"/>
-    <geometry>
-      <mesh filename="package://swarm/meshes/bumper.dae" scale="1 1 1"/>
-    </geometry>
-    <material name="black">
+      </visual>
+      <visual name="front_bumper_visual">
+        <origin xyz="0.48 0 0.091" rpy="0 0 0"/>
+        <geometry>
+          <mesh filename="package://swarm/meshes/bumper.dae"/>
+        </geometry>
+        <material name="black">
           <color rgba="0.1 0.1 0.1 1"/>
         </material>
-  </visual>
-  <visual name="rear_bumper_visual">
-    <origin xyz="-0.48 0 0.091" rpy="0 0 3.14159"/>
-    <geometry>
-      <mesh filename="package://swarm/meshes/bumper.dae" scale="1 1 1"/>
-    </geometry>
-    <material name="black">
+      </visual>
+      <visual name="rear_bumper_visual">
+        <origin xyz="-0.48 0 0.091" rpy="0 0 3.14159"/>
+        <geometry>
+          <mesh filename="package://swarm/meshes/bumper.dae"/>
+        </geometry>
+        <material name="black">
           <color rgba="0.1 0.1 0.1 1"/>
         </material>
-  </visual>
-    <visual name="top_chassis_visual">
-    <origin xyz="0 0 0" rpy="0 0 0"/>
-    <geometry>
-      <mesh filename="package://swarm/meshes/top_chassis.stl" scale="1 1 1"/>
-    </geometry>
-    <material name="teal">
+      </visual>
+      <visual name="top_chassis_visual">
+        <geometry>
+          <mesh filename="package://swarm/meshes/top_chassis.stl"/>
+        </geometry>
+        <material name="teal">
           <color rgba="0 0.5 0.5 1"/>
         </material>
-  </visual>
-  <visual name="lidar_base_visual">
-  <origin xyz="0.424 0 0.327" rpy="0 0 0"/>
-  <geometry>
-  	<mesh filename="package://swarm/meshes/VLP16_base_1.dae" scale="1 1 1"/>
-  </geometry>
-  </visual>
-    <visual name="lidar_base_visual_2">
-  <origin xyz="0.424 0 0.327" rpy="0 0 0"/>
-  <geometry>
-  	<mesh filename="package://swarm/meshes/VLP16_base_2.dae" scale="1 1 1"/>
-  </geometry>
-  </visual>
-      <visual name="lidar_scan_visual">
-  <origin xyz="0.424 0 0.327" rpy="0 0 0"/>
-  <geometry>
-  	<mesh filename="package://swarm/meshes/VLP16_scan.dae" scale="1 1 1"/>
-  </geometry>
-  </visual>
+      </visual>
       <visual name="user_rail_visual">
-  <origin xyz="0.272 0 0.245" rpy="0 0 0"/>
-  <geometry>
-  	<mesh filename="package://swarm/meshes/user_rail.dae" scale="1 1 1"/>
-  </geometry>
-  <material name="black">
-  	<color rgba="0.1 0.1 0.1 1"/>
-  </material>
-  </visual>
-        <visual name="holder_visual">
-  <origin xyz="0.272 0 0" rpy="0 0 0"/>
-  <geometry>
-  	<mesh filename="package://swarm/meshes/holder.stl" scale="1 1 1"/>
-  </geometry>
-  <material name="black">
-  	<color rgba="0.1 0.1 0.1 1"/>
-  </material>
-  </visual>
-</link>
-<joint name="base_link_joint" type="fixed">
-  <parent link="base_link"/>
-  <child link="ground_bot_frame"/>
-  <origin xyz="0 0 0" rpy="0 0 0"/>
-</joint>
-<!-- My Sensors -->
-<gazebo reference="base_link">
+        <origin xyz="0.272 0 0.245" rpy="0 0 0"/>
+        <geometry>
+          <mesh filename="package://swarm/meshes/user_rail.dae"/>
+        </geometry>
+        <material name="black">
+          <color rgba="0.1 0.1 0.1 1"/>
+        </material>
+      </visual>
+    </link>
+    <joint name="base_link_joint" type="fixed">
+      <parent link="base_link"/>
+      <child link="ground_bot_frame"/>
+      <origin xyz="0 0 0" rpy="0 0 0"/>
+    </joint>
+    <gazebo reference="ground_bot_frame">
       <sensor name="imu_sensor" type="imu">
         <always_on>true</always_on>
-        <update_rate>10</update_rate>
+        <update_rate>100</update_rate>
         <visualize>true</visualize>
         <topic>imu</topic>
       </sensor>
-</gazebo>
-</xacro:macro>
+    </gazebo>
+  </xacro:macro>
 </robot>

File: src/swarm/model/robot.xacro (robot description, xacro)
@@ -1,18 +1,30 @@
-<?xml version="1.0"?>
-<robot xmlns:xacro="http://www.ros.org/wiki/xacro" name="Ground_bot">
+<?xml version="1.9"?>
+<robot
+  xmlns:xacro="http://www.ros.org/wiki/xacro"
+  name="Ground_bot">
+  <!-- Main frame -->
   <xacro:include filename="$(find swarm)/model/main_frame.xacro"/>
   <xacro:bot/>
+  <!-- Wheels -->
   <xacro:include filename="$(find swarm)/model/wheels.xacro"/>
   <xacro:wheels/>
+  <!-- Cameras -->
   <xacro:include filename="cameras.xacro"/>
   <xacro:depth_camera
-    name="front_camera_link"
+    name="front_camera"
     parent="ground_bot_frame"
     xyz="0.478 0 0.285"
     rpy="0 0 0"/>
   <xacro:depth_camera
-    name="down_camera_link"
+    name="down_camera"
     parent="ground_bot_frame"
     xyz="0.478 0 0.200"
     rpy="0 0.5236 0"/>
+  <!-- LiDAR -->
+  <xacro:include filename="$(find swarm)/model/lidar.xacro"/>
+  <xacro:lidar
+    name="lidar"
+    parent="ground_bot_frame"
+    xyz="0.424 0 0.327"
+    rpy="0 0 0"/>
 </robot>

File: src/swarm/model/wheels.xacro (robot description, xacro)
@@ -1,3 +1,3 @@
-<?xml version="1.0"?>
+<?xml version="1.9"?>
 <robot xmlns:xacro="http://www.ros.org/wiki/xacro">
   <xacro:macro name="wheel_link" params="name mesh scale mass ixx iyy izz">

Commit message: multi_ground_bot spawned

File: src/swarm/model/cameras.xacro (robot description, xacro)
@@ -1,6 +1,6 @@
-<?xml version="1.9"?>
+<?xml version="1.0"?>
 <robot xmlns:xacro="http://www.ros.org/wiki/xacro">
-  <xacro:macro name="depth_camera" params="name parent xyz rpy">
-    <link name="${name}">
+  <xacro:macro name="depth_camera" params="name parent xyz rpy suffix">
+    <link name="${suffix}${name}">
       <visual>
         <geometry>
@@ -27,16 +27,16 @@
       </inertial>
     </link>
-    <joint name="${name}_joint" type="fixed">
+    <joint name="${suffix}${name}_joint" type="fixed">
       <parent link="${parent}"/>
-      <child link="${name}"/>
+      <child link="${suffix}${name}"/>
       <origin xyz="${xyz}" rpy="${rpy}"/>
     </joint>
-    <gazebo reference="${name}">
-      <sensor name="${name}_sensor" type="rgbd_camera">
+    <gazebo reference="${suffix}${name}">
+      <sensor name="${suffix}${name}_sensor" type="rgbd_camera">
         <always_on>true</always_on>
         <update_rate>30</update_rate>
         <visualize>true</visualize>
-        <ignition_frame_id>${name}</ignition_frame_id>
         <topic>${name}</topic>
+        <ignition_frame_id>${suffix}${name}</ignition_frame_id>
         <camera>
           <horizontal_fov>1.92</horizontal_fov>

File: src/swarm/model/drone.xacro (robot description, xacro)
@@ -1,6 +1,6 @@
-<?xml version="1.9"?>
-<robot xmlns:xacro="http://www.ros.org/wiki/xacro">
+<?xml version="1.0"?>
+<robot xmlns:xacro="http://www.ros.org/wiki/xacro" name="drone">
   <xacro:macro name="drone">
-    <link name="drone_base_link"/>
+    <link name="base_link"/>
     <link name="drone_frame">
       <inertial>
@@ -31,5 +31,5 @@
     </link>
     <joint name="drone_base_link_joint" type="fixed">
-      <parent link="drone_base_link"/>
+      <parent link="base_link"/>
       <child link="drone_frame"/>
       <origin xyz="1.0 0" rpy="0 0 0"/>

File: src/swarm/model/ground_bot.xacro (robot description, xacro)
@@ -1,7 +1,7 @@
-<?xml version="1.9"?>
+<?xml version="1.0"?>
 <robot xmlns:xacro="http://www.ros.org/wiki/xacro">
-  <xacro:macro name="ground_bot">
-    <link name="base_link"/>
-    <link name="ground_bot_frame">
+  <xacro:macro name="ground_bot" params="suffix">
+    <link name="${suffix}base_link"/>
+    <link name="${suffix}ground_bot_frame">
       <inertial>
         <origin xyz="0.0 0.0 -0.25" rpy="0 0 0"/>
@@ -27,43 +27,7 @@
         </geometry>
       </collision>
-      <collision name="frame_collision_1">
-        <origin xyz="0 0 0.185625" rpy="0 0 0"/>
-        <geometry>
-          <box size="0.78992 0.5709 0.12375"/>
-        </geometry>
-      </collision>
-            <collision name="top_chassis_collision">
-        <origin xyz="0 0 0" rpy="0 0 0"/>
-        <geometry>
-          <box size="0.0078 0.13 0.0192"/>
-        </geometry>
-      </collision>
-      <collision name="user_rail_collision">
-        <origin xyz="0.272 0 0.245" rpy="0 0 0"/>
-        <geometry>
-          <box size="0.0078 0.13 0.0192"/>
-        </geometry>
-      </collision>
       <visual name="main_frame_visual">
         <geometry>
           <mesh filename="package://swarm/meshes/main_frame.stl"/>
-        </geometry>
-        <material name="black">
-          <color rgba="0.1 0.1 0.1 1"/>
-        </material>
-      </visual>
-      <visual name="front_bumper_visual">
-        <origin xyz="0.48 0 0.091" rpy="0 0 0"/>
-        <geometry>
-          <mesh filename="package://swarm/meshes/bumper.dae"/>
-        </geometry>
-        <material name="black">
-          <color rgba="0.1 0.1 0.1 1"/>
-        </material>
-      </visual>
-      <visual name="rear_bumper_visual">
-        <origin xyz="-0.48 0 0.091" rpy="0 0 3.14159"/>
-        <geometry>
-          <mesh filename="package://swarm/meshes/bumper.dae"/>
         </geometry>
         <material name="black">
@@ -79,20 +43,11 @@
         </material>
       </visual>
-      <visual name="user_rail_visual">
-        <origin xyz="0.272 0 0.245" rpy="0 0 0"/>
-        <geometry>
-          <mesh filename="package://swarm/meshes/user_rail.dae"/>
-        </geometry>
-        <material name="black">
-          <color rgba="0.1 0.1 0.1 1"/>
-        </material>
-      </visual>
     </link>
-    <joint name="base_link_joint" type="fixed">
-      <parent link="base_link"/>
-      <child link="ground_bot_frame"/>
+    <joint name="${suffix}base_link_joint" type="fixed">
+      <parent link="${suffix}base_link"/>
+      <child link="${suffix}ground_bot_frame"/>
       <origin xyz="0 0 0" rpy="0 0 0"/>
     </joint>
-    <gazebo reference="ground_bot_frame">
+    <gazebo reference="${suffix}ground_bot_frame">
       <sensor name="imu" type="imu">
         <always_on>true</always_on>

File: src/swarm/model/lidar.xacro (robot description, xacro)
@@ -1,6 +1,6 @@
-<?xml version="1.9"?>
+<?xml version="1.0"?>
 <robot xmlns:xacro="http://www.ros.org/wiki/xacro">
-  <xacro:macro name="lidar" params="name parent xyz rpy">
-    <link name="${name}">
+  <xacro:macro name="lidar" params="name parent xyz rpy suffix">
+    <link name="${suffix}${name}">
       <visual name="lidar_base_visual_2">
         <origin xyz="0 0 0" rpy="0 0 0"/>
@@ -36,5 +36,5 @@
         <origin xyz="0.212 0 0.164" rpy="0 0 0"/>
         <geometry>
-          <mesh size="0.0078 0.13 0.0192"/>
+          <box size="0.0078 0.13 0.0192"/>
         </geometry>
       </collision>
@@ -45,15 +45,16 @@
       </collision>
     </link>
-    <joint name="${name}_joint" type="fixed">
+    <joint name="${suffix}${name}_joint" type="fixed">
       <parent link="${parent}"/>
-      <child link="${name}"/>
+      <child link="${suffix}${name}"/>
       <origin xyz="${xyz}" rpy="${rpy}"/>
     </joint>
-    <gazebo reference="${name}">
-      <sensor name="${name}_lidar" type="gpu_lidar">
+    <gazebo reference="${suffix}${name}">
+      <sensor name="${suffix}${name}_lidar" type="gpu_lidar">
         <always_on>true</always_on>
         <update_rate>30</update_rate>
         <visualize>true</visualize>
-        <frame_id>${name}</frame_id>
+        <topic>lidar/points</topic>
+        <frame_id>${suffix}${name}</frame_id>
         <lidar>
           <scan>

File: src/swarm/model/robot.xacro (robot description, xacro)
@@ -1,29 +1,17 @@
-<?xml version="1.9"?>
-<robot
-  xmlns:xacro="http://www.ros.org/wiki/xacro"
-  name="Ground_bot">
+<?xml version="1.0"?>
+<robot xmlns:xacro="http://www.ros.org/wiki/xacro" name="Ground_bot">
+  <xacro:arg name="frame_prefix" default=""/>
   <xacro:include filename="$(find swarm)/model/robot.gazebo"/>
-  <!-- Ground Bot -->
   <xacro:include filename="$(find swarm)/model/ground_bot.xacro"/>
-  <xacro:ground_bot/>
-    <!-- Drone
-  <xacro:include filename="$(find swarm)/model/drone.xacro"/>
--->
-  <!-- Wheels -->
   <xacro:include filename="$(find swarm)/model/wheels.xacro"/>
-  <xacro:wheels/>
-  <!-- Cameras -->
-  <xacro:include filename="cameras.xacro"/>
-  <xacro:depth_camera
-    name="front_camera"
-    parent="ground_bot_frame"
-    xyz="0.478 0 0.285"
-    rpy="0 0 0"/>
-  <!-- LiDAR -->
   <xacro:include filename="$(find swarm)/model/lidar.xacro"/>
+  <xacro:include filename="$(find swarm)/model/cameras.xacro"/>
+  <xacro:ground_bot suffix="$(arg frame_prefix)"/>
+  <xacro:wheels suffix="$(arg frame_prefix)"/>
   <xacro:lidar
     name="lidar"
-    parent="ground_bot_frame"
+    parent="$(arg frame_prefix)ground_bot_frame"
     xyz="0.424 0 0.327"
-    rpy="0 0 0"/>
+    rpy="0 0 0"
+    suffix="$(arg frame_prefix)"/>
 </robot>

File: src/swarm/model/wheels.xacro (robot description, xacro)
@@ -1,3 +1,3 @@
-<?xml version="1.9"?>
+<?xml version="1.0"?>
 <robot xmlns:xacro="http://www.ros.org/wiki/xacro">
   <xacro:macro name="wheel_link" params="name mesh scale mass ixx iyy izz">
@@ -29,37 +29,36 @@
     </link>
   </xacro:macro>
-  <xacro:macro name="wheels">
-    <xacro:wheel_link name="front_left_wheel"  mesh="wheel.stl" scale="1 1 1"
+  <xacro:macro name="wheels" params="suffix">
+    <xacro:wheel_link name="${suffix}front_left_wheel"  mesh="wheel.stl" scale="1 1 1"
                       mass="2.637" ixx="0.0246" iyy="0.04411" izz="0.0246"/>
-    <xacro:wheel_link name="front_right_wheel" mesh="wheel.stl" scale="1 1 1"
+    <xacro:wheel_link name="${suffix}front_right_wheel" mesh="wheel.stl" scale="1 1 1"
                       mass="2.637" ixx="0.0246" iyy="0.04411" izz="0.0246"/>
-    <xacro:wheel_link name="rear_left_wheel"   mesh="wheel.stl" scale="1 1 1"
+    <xacro:wheel_link name="${suffix}rear_left_wheel"   mesh="wheel.stl" scale="1 1 1"
                       mass="2.637" ixx="0.0246" iyy="0.04411" izz="0.0246"/>
-    <xacro:wheel_link name="rear_right_wheel"  mesh="wheel.stl" scale="1 1 1"
+    <xacro:wheel_link name="${suffix}rear_right_wheel"  mesh="wheel.stl" scale="1 1 1"
                       mass="2.637" ixx="0.0246" iyy="0.04411" izz="0.0246"/>
-    <joint name="front_left_wheel_joint" type="revolute">
-      <parent link="base_link"/>
-      <child link="front_left_wheel"/>
+    <joint name="${suffix}front_left_wheel_joint" type="revolute">
+      <parent link="${suffix}base_link"/>  <child link="${suffix}front_left_wheel"/>
       <origin xyz="0.256 0.2854 0.03282" rpy="0 0 0"/>
       <axis xyz="0 1 0"/>
       <limit lower="-1e16" upper="1e16" effort="20" velocity="50"/>
     </joint>
-    <joint name="front_right_wheel_joint" type="revolute">
-      <parent link="base_link"/>
-      <child link="front_right_wheel"/>
+    <joint name="${suffix}front_right_wheel_joint" type="revolute">
+      <parent link="${suffix}base_link"/>
+      <child link="${suffix}front_right_wheel"/>
       <origin xyz="0.256 -0.2854 0.03282" rpy="0 0 0"/>
       <axis xyz="0 1 0"/>
       <limit lower="-1e16" upper="1e16" effort="20" velocity="50"/>
     </joint>
-    <joint name="rear_left_wheel_joint" type="revolute">
-      <parent link="base_link"/>
-      <child link="rear_left_wheel"/>
+    <joint name="${suffix}rear_left_wheel_joint" type="revolute">
+      <parent link="${suffix}base_link"/>
+      <child link="${suffix}rear_left_wheel"/>
       <origin xyz="-0.256 0.2854 0.03282" rpy="0 0 0"/>
       <axis xyz="0 1 0"/>
       <limit lower="-1e16" upper="1e16" effort="20" velocity="50"/>
     </joint>
-    <joint name="rear_right_wheel_joint" type="revolute">
-      <parent link="base_link"/>
-      <child link="rear_right_wheel"/>
+    <joint name="${suffix}rear_right_wheel_joint" type="revolute">
+      <parent link="${suffix}base_link"/>
+      <child link="${suffix}rear_right_wheel"/>
       <origin xyz="-0.256 -0.2854 0.03282" rpy="0 0 0"/>
       <axis xyz="0 1 0"/>
