Commit message: stable drone + drone teleop

File: src/swarm/model/cameras.xacro (robot description, xacro)
@@ -4,25 +4,13 @@
     <link name="${suffix}${name}">
       <visual>
-        <geometry>
-          <mesh filename="package://swarm/meshes/zed2i.stl"/>
-        </geometry>
-        <material name="grey">
-          <color rgba="0.2 0.2 0.2 1"/>
-        </material>
+        <geometry><mesh filename="package://swarm/meshes/zed2i.stl"/></geometry>
+        <material name="grey"><color rgba="0.2 0.2 0.2 1"/></material>
       </visual>
       <collision>
-        <geometry>
-          <mesh filename="package://swarm/meshes/zed2i.stl"/>
-        </geometry>
+        <geometry><mesh filename="package://swarm/meshes/zed2i.stl"/></geometry>
       </collision>
       <inertial>
         <mass value="0.05"/>
-        <inertia
-          ixx="0.0001"
-          ixy="0"
-          ixz="0"
-          iyy="0.0001"
-          iyz="0"
-          izz="0.0001"/>
+        <inertia ixx="0.0001" ixy="0" ixz="0" iyy="0.0001" iyz="0" izz="0.0001"/>
       </inertial>
     </link>
@@ -33,35 +21,23 @@
     </joint>
     <gazebo reference="${suffix}${name}">
-      <sensor name="${suffix}${name}_sensor" type="rgbd_camera">
+      <sensor name="depth_camera" type="rgbd_camera">
         <always_on>true</always_on>
         <update_rate>30</update_rate>
         <visualize>true</visualize>
-        <topic>${name}</topic>
+        <topic>camera</topic>
         <ignition_frame_id>${suffix}${name}</ignition_frame_id>
         <camera>
           <horizontal_fov>1.92</horizontal_fov>
-          <image>
-            <width>1280</width>
-            <height>720</height>
-            <format>R8G8B8</format>
-          </image>
-          <clip>
-            <near>0.2</near>
-            <far>20.0</far>
-          </clip>
-          <noise>
-            <type>gaussian</type>
-            <mean>0.0</mean>
-            <stddev>0.002</stddev>
-          </noise>
+          <image><width>640</width><height>480</height><format>R8G8B8</format></image>
+          <clip><near>0.2</near><far>20.0</far></clip>
         </camera>
-        <depth_camera>
-          <clip>
-            <near>0.2</near>
-            <far>20.0</far>
-          </clip>
-        </depth_camera>
       </sensor>
     </gazebo>
   </xacro:macro>
+    <xacro:depth_camera
+    name="depth_camera"
+    parent="$(arg frame_prefix)ground_bot_frame"
+    xyz="0.424 0 0.5"
+    rpy="0 0 0"
+    suffix="$(arg frame_prefix)"/>
 </robot>

File: src/swarm/model/drone.xacro (robot description, xacro)
@@ -16,5 +16,5 @@
       </inertial>
       <collision name="drone_frame_collision">
-        <origin xyz="-0.00424 0.00014 -0.00595" rpy="0 0 0"/>
+        <origin xyz="0.0 0.0 0.0" rpy="0 0 0"/>
         <geometry>
           <box size="0.316618 0.330564 0.089582"/>

File: src/swarm/model/propellers.xacro (robot description, xacro)
@@ -15,7 +15,5 @@
           <mesh filename="file://$(find swarm)/meshes/${mesh}" scale="${scale}"/>
         </geometry>
-        <material name="black">
-          <color rgba="0.1 0.1 0.1 1"/>
-        </material>
+        <material name="black"><color rgba="0.1 0.1 0.1 1"/></material>
       </visual>
     </link>
@@ -27,5 +25,5 @@
       scale="1 1 1"
       mass="0.005"
-      ixx="0.00043333" iyy="0.00043333" izz="0.0008"/>
+      ixx="0.00001" iyy="0.00001" izz="0.00002"/>
     <xacro:propeller_link
       name="front_right_propeller"
@@ -33,5 +31,5 @@
       scale="1 1 1"
       mass="0.005"
-      ixx="0.00043333" iyy="0.00043333" izz="0.0008"/>
+      ixx="0.00001" iyy="0.00001" izz="0.00002"/>
     <xacro:propeller_link
       name="rear_right_propeller"
@@ -39,5 +37,5 @@
       scale="1 1 1"
       mass="0.005"
-      ixx="0.00043333" iyy="0.00043333" izz="0.0008"/>
+      ixx="0.00001" iyy="0.00001" izz="0.00002"/>
     <xacro:propeller_link
       name="rear_left_propeller"
@@ -45,9 +43,9 @@
       scale="1 1 1"
       mass="0.005"
-      ixx="0.00043333" iyy="0.00043333" izz="0.0008"/>
+      ixx="0.00001" iyy="0.00001" izz="0.00002"/>
     <joint name="front_right_propeller_joint" type="continuous">
       <parent link="drone_base_link"/>
       <child link="front_right_propeller"/>
-      <origin xyz="0.08456 -0.11435 -0.00501" rpy="0 0 0"/>
+      <origin xyz="0.09 -0.115 -0.005" rpy="0 0 0"/>
       <axis xyz="0 0 1"/>
     </joint>
@@ -55,5 +53,5 @@
       <parent link="drone_base_link"/>
       <child link="front_left_propeller"/>
-      <origin xyz="0.08456 0.11463 -0.00501" rpy="0 0 0"/>
+      <origin xyz="0.09 0.115 -0.005" rpy="0 0 0"/>
       <axis xyz="0 0 1"/>
     </joint>
@@ -61,5 +59,5 @@
       <parent link="drone_base_link"/>
       <child link="rear_right_propeller"/>
-      <origin xyz="-0.09035 -0.11423 -0.00501" rpy="0 0 0"/>
+      <origin xyz="-0.09 -0.115 -0.005" rpy="0 0 0"/>
       <axis xyz="0 0 1"/>
     </joint>
@@ -67,5 +65,5 @@
       <parent link="drone_base_link"/>
       <child link="rear_left_propeller"/>
-      <origin xyz="-0.09035 0.11452 -0.00501" rpy="0 0 0"/>
+      <origin xyz="-0.09 0.115 -0.005" rpy="0 0 0"/>
       <axis xyz="0 0 1"/>
     </joint>
