Commit message: drone flying

File: src/swarm/model/drone.xacro (robot description, xacro)
@@ -1,17 +1,17 @@
 <?xml version="1.0"?>
 <robot xmlns:xacro="http://www.ros.org/wiki/xacro" name="drone">
-  <xacro:macro name="drone">
-    <link name="base_link"/>
-    <link name="drone_frame">
+  <xacro:macro name="drone_macro" params="">
+    <link name="drone_base_link"/>
+<link name="drone_frame">
       <inertial>
-        <origin xyz="1.0 0.0 0.0" rpy="0 0 0"/>
-        <mass value="2.0"/>
+        <origin xyz="0.0 0.0 0.0" rpy="0 0 0"/>
+        <mass value="1.503"/>
         <inertia
-          ixx="1.805e-3"
-          ixy="-8.619e-7"
-          ixz="1.764e-3"
-          iyy="1.555e-5"
-          iyz="3.595e-7"
-          izz="3.328e-3"/>
+          ixx="0.02"
+          ixy="0.0"
+          ixz="0.0"
+          iyy="0.02"
+          iyz="0.0"
+          izz="0.04"/>
       </inertial>
       <collision name="drone_frame_collision">
@@ -26,14 +26,13 @@
         </geometry>
         <material name="black">
-          <color rgba="0.1 0.1 0.1 1"/>
+          <color rgba="1 0.35 0.12 1"/>
         </material>
       </visual>
     </link>
     <joint name="drone_base_link_joint" type="fixed">
-      <parent link="base_link"/>
+      <parent link="drone_base_link"/>
       <child link="drone_frame"/>
-      <origin xyz="1.0 0" rpy="0 0 0"/>
+      <origin xyz="0 0 0" rpy="0 0 0"/>
     </joint>
   </xacro:macro>
-    <xacro:drone/>
 </robot>

Commit message: docs: adjust README structure and finalize drone xacro namespacing
- ReadMe.md: revert to simple list structure for project directories and restore original overview text.
- drone.gazebo, drone.xacro, propellers.xacro, robot_drone.xacro: add support for frame_prefix and robot_ns arguments to properly isolate links, joints, and Gazebo plugin namespaces across multiple spawned drones.

File: src/swarm/model/drone.xacro (robot description, xacro)
@@ -1,19 +1,16 @@
 <?xml version="1.0"?>
 <robot xmlns:xacro="http://www.ros.org/wiki/xacro" name="drone">
-  <xacro:macro name="drone_macro" params="">
-    <link name="drone_base_link"/>
-<link name="drone_frame">
+  <xacro:macro name="drone_macro" params="suffix">
+    <link name="${suffix}drone_base_link"/>
+    <link name="${suffix}drone_frame">
       <inertial>
         <origin xyz="0.0 0.0 0.0" rpy="0 0 0"/>
         <mass value="1.503"/>
         <inertia
-          ixx="0.02"
-          ixy="0.0"
-          ixz="0.0"
-          iyy="0.02"
-          iyz="0.0"
+          ixx="0.02" ixy="0.0" ixz="0.0"
+          iyy="0.02" iyz="0.0"
           izz="0.04"/>
       </inertial>
-      <collision name="drone_frame_collision">
+      <collision name="${suffix}drone_frame_collision">
         <origin xyz="0.0 0.0 0.0" rpy="0 0 0"/>
         <geometry>
@@ -21,5 +18,5 @@
         </geometry>
       </collision>
-      <visual name="drone_frame_visual">
+      <visual name="${suffix}drone_frame_visual">
         <geometry>
           <mesh filename="package://swarm/meshes/hull.dae"/>
@@ -30,7 +27,7 @@
       </visual>
     </link>
-    <joint name="drone_base_link_joint" type="fixed">
-      <parent link="drone_base_link"/>
-      <child link="drone_frame"/>
+    <joint name="${suffix}drone_base_link_joint" type="fixed">
+      <parent link="${suffix}drone_base_link"/>
+      <child link="${suffix}drone_frame"/>
       <origin xyz="0 0 0" rpy="0 0 0"/>
     </joint>

File: src/swarm/model/propellers.xacro (robot description, xacro)
@@ -13,5 +13,5 @@
       <visual>
         <geometry>
-          <mesh filename="file://$(find swarm)/meshes/${mesh}" scale="${scale}"/>
+          <mesh filename="package://swarm/meshes/${mesh}" scale="${scale}"/>
         </geometry>
         <material name="black"><color rgba="0.1 0.1 0.1 1"/></material>
@@ -19,50 +19,42 @@
     </link>
   </xacro:macro>
-  <xacro:macro name="propellers">
+  <xacro:macro name="propellers" params="suffix">
     <xacro:propeller_link
-      name="front_left_propeller"
-      mesh="propeller_fl.dae"
-      scale="1 1 1"
-      mass="0.005"
-      ixx="0.00001" iyy="0.00001" izz="0.00002"/>
+      name="${suffix}front_left_propeller"
+      mesh="propeller_fl.dae" scale="1 1 1"
+      mass="0.005" ixx="0.00001" iyy="0.00001" izz="0.00002"/>
     <xacro:propeller_link
-      name="front_right_propeller"
-      mesh="propeller_fr.dae"
-      scale="1 1 1"
-      mass="0.005"
-      ixx="0.00001" iyy="0.00001" izz="0.00002"/>
+      name="${suffix}front_right_propeller"
+      mesh="propeller_fr.dae" scale="1 1 1"
+      mass="0.005" ixx="0.00001" iyy="0.00001" izz="0.00002"/>
     <xacro:propeller_link
-      name="rear_right_propeller"
-      mesh="propeller_rr.dae"
-      scale="1 1 1"
-      mass="0.005"
-      ixx="0.00001" iyy="0.00001" izz="0.00002"/>
+      name="${suffix}rear_right_propeller"
+      mesh="propeller_rr.dae" scale="1 1 1"
+      mass="0.005" ixx="0.00001" iyy="0.00001" izz="0.00002"/>
     <xacro:propeller_link
-      name="rear_left_propeller"
-      mesh="propeller_rl.dae"
-      scale="1 1 1"
-      mass="0.005"
-      ixx="0.00001" iyy="0.00001" izz="0.00002"/>
-    <joint name="front_right_propeller_joint" type="continuous">
-      <parent link="drone_base_link"/>
-      <child link="front_right_propeller"/>
+      name="${suffix}rear_left_propeller"
+      mesh="propeller_rl.dae" scale="1 1 1"
+      mass="0.005" ixx="0.00001" iyy="0.00001" izz="0.00002"/>
+    <joint name="${suffix}front_right_propeller_joint" type="continuous">
+      <parent link="${suffix}drone_base_link"/>
+      <child link="${suffix}front_right_propeller"/>
       <origin xyz="0.09 -0.115 -0.005" rpy="0 0 0"/>
       <axis xyz="0 0 1"/>
     </joint>
-    <joint name="front_left_propeller_joint" type="continuous">
-      <parent link="drone_base_link"/>
-      <child link="front_left_propeller"/>
+    <joint name="${suffix}front_left_propeller_joint" type="continuous">
+      <parent link="${suffix}drone_base_link"/>
+      <child link="${suffix}front_left_propeller"/>
       <origin xyz="0.09 0.115 -0.005" rpy="0 0 0"/>
       <axis xyz="0 0 1"/>
     </joint>
-    <joint name="rear_right_propeller_joint" type="continuous">
-      <parent link="drone_base_link"/>
-      <child link="rear_right_propeller"/>
+    <joint name="${suffix}rear_right_propeller_joint" type="continuous">
+      <parent link="${suffix}drone_base_link"/>
+      <child link="${suffix}rear_right_propeller"/>
       <origin xyz="-0.09 -0.115 -0.005" rpy="0 0 0"/>
       <axis xyz="0 0 1"/>
     </joint>
-    <joint name="rear_left_propeller_joint" type="continuous">
-      <parent link="drone_base_link"/>
-      <child link="rear_left_propeller"/>
+    <joint name="${suffix}rear_left_propeller_joint" type="continuous">
+      <parent link="${suffix}drone_base_link"/>
+      <child link="${suffix}rear_left_propeller"/>
       <origin xyz="-0.09 0.115 -0.005" rpy="0 0 0"/>
       <axis xyz="0 0 1"/>

File: src/swarm/model/robot_drone.xacro (robot description, xacro)
@@ -1,9 +1,12 @@
 <?xml version="1.0"?>
 <robot xmlns:xacro="http://www.ros.org/wiki/xacro" name="drone">
+  <xacro:arg name="frame_prefix" default=""/>
+  <xacro:arg name="robot_ns" default="drone"/>
   <xacro:include filename="$(find swarm)/model/drone.gazebo"/>
   <xacro:include filename="$(find swarm)/model/drone.xacro"/>
   <xacro:include filename="$(find swarm)/model/propellers.xacro"/>
-  <xacro:drone_macro />
-  <xacro:propellers/>
-  <xacro:drone_gazebo suffix=""/>
+  <xacro:drone_macro suffix="$(arg frame_prefix)"/>
+  <xacro:propellers suffix="$(arg frame_prefix)"/>
+  <!-- robot_ns controls Gazebo topic namespace; suffix controls link/joint names -->
+  <xacro:drone_gazebo suffix="$(arg frame_prefix)" robot_ns="$(arg robot_ns)"/>
 </robot>
